File: hw/fh07_node/power_converter.kicad_sch (KiCad schematic)
At the start: 7 parts

Commit message: Completed hardware revision 1 release
Parts:
- added J2: Conn_01x02, Connector_Molex:Molex_Micro-Fit_3.0_43650-0221_1x02_P3.00mm_Vertical, symbol Connector_Generic:Conn_01x02
- C1, C2, C3, C4, C5, C6, C7: footprint (none) -> Capacitor_SMD:C_1206_3216Metric_Pad1.33x1.80mm_HandSolder
Connections:
- net +2V5: now also J2.2 (Pin_2)
- net GND: now also J2.1 (Pin_1)
