File: hw/fh07_node/sensors.kicad_sch (KiCad schematic)
At the start: 8 parts, among them U1 BNO055

Commit message: Completed hardware revision 1 release
Parts:
- C10: renamed from C2; footprint (none) -> Capacitor_SMD:C_1206_3216Metric_Pad1.33x1.80mm_HandSolder
- C11: renamed from C3; footprint (none) -> Capacitor_SMD:C_1206_3216Metric_Pad1.33x1.80mm_HandSolder
- C12: renamed from C1; footprint (none) -> Capacitor_SMD:C_1206_3216Metric_Pad1.33x1.80mm_HandSolder
- R_PULL1: renamed from R_PULL3; footprint (none) -> Resistor_SMD:R_1206_3216Metric_Pad1.30x1.75mm_HandSolder
- R_PULL2: renamed from R_PULL4; footprint (none) -> Resistor_SMD:R_1206_3216Metric_Pad1.30x1.75mm_HandSolder
- R_PULL3: renamed from R_PULL2; footprint (none) -> Resistor_SMD:R_1206_3216Metric_Pad1.30x1.75mm_HandSolder
- R_PULL4: renamed from R_PULL1; footprint (none) -> Resistor_SMD:R_1206_3216Metric_Pad1.30x1.75mm_HandSolder
- U1: footprint BNO055:LGA28R50P4X10_380X520X100 -> ProjectFootprintLib:LGA28R50P4X10_380X520X100
Changed lines of the file:
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@@
 		(dnp no)
 		(fields_autoplaced yes)
-		(property "Reference" "C2"
+		(property "Reference" "C10"
 			(at 100.33 114.2999 0)
 			(effects
@@
 			)
 		)
-		(property "Footprint" ""
+		(property "Footprint" "Capacitor_SMD:C_1206_3216Metric_Pad1.33x1.80mm_HandSolder"
 			(at 97.4852 119.38 0)
 			(effects
@@
 				)
 			)
+			(project "fh07_node"
+				(path "/aea54c0a-0593-4c80-97cc-583e63973e87/f7042617-bbaf-4506-802a-37539c441d1d"
+					(reference "C10")
+					(unit 1)
+				)
+			)
 		)
 	)
@@
 		(dnp no)
 		(fields_autoplaced yes)
-		(property "Reference" "#PWR07"
+		(property "Reference" "#PWR0113"
 			(at 96.52 128.27 0)
 			(effects
@@
 				)
 			)
+			(project "fh07_node"
+				(path "/aea54c0a-0593-4c80-97cc-583e63973e87/f7042617-bbaf-4506-802a-37539c441d1d"
+					(reference "#PWR0113")
+					(unit 1)
+				)
+			)
 		)
 	)
@@
 		(on_board yes)
 		(dnp no)
-		(property "Reference" "R_PULL1"
+		(property "Reference" "R_PULL4"
 			(at 86.614 110.998 0)
 			(effects
@@
 			)
 		)
-		(property "Footprint" ""
+		(property "Footprint" "Resistor_SMD:R_1206_3216Metric_Pad1.30x1.75mm_HandSolder"
 			(at 82.042 113.03 90)
 			(effects
@@
 				)
 			)
+			(project "fh07_node"
+				(path "/aea54c0a-0593-4c80-97cc-583e63973e87/f7042617-bbaf-4506-802a-37539c441d1d"
+					(reference "R_PULL4")
+					(unit 1)
+				)
+			)
 		)
 	)
@@
 		(on_board yes)
 		(dnp no)
-		(property "Reference" "R_PULL2"
+		(property "Reference" "R_PULL3"
 			(at 86.106 100.584 0)
 			(effects
@@
 			)
 		)
-		(property "Footprint" ""
+		(property "Footprint" "Resistor_SMD:R_1206_3216Metric_Pad1.30x1.75mm_HandSolder"
 			(at 82.042 102.87 90)
 			(effects
@@
 				)
 			)
+			(project "fh07_node"
+				(path "/aea54c0a-0593-4c80-97cc-583e63973e87/f7042617-bbaf-4506-802a-37539c441d1d"
+					(reference "R_PULL3")
+					(unit 1)
+				)
+			)
 		)
 	)
@@
 		(dnp no)
 		(fields_autoplaced yes)
-		(property "Reference" "C1"
+		(property "Reference" "C12"
 			(at 173.99 96.5199 0)
 			(effects
@@
 			)
 		)
-		(property "Footprint" ""
+		(property "Footprint" "Capacitor_SMD:C_1206_3216Metric_Pad1.33x1.80mm_HandSolder"
 			(at 171.1452 101.6 0)
 			(effects
@@
 				)
 			)
+			(project "fh07_node"
+				(path "/aea54c0a-0593-4c80-97cc-583e63973e87/f7042617-bbaf-4506-802a-37539c441d1d"
+					(reference "C12")
+					(unit 1)
+				)
+			)
 		)
 	)
@@
 		(dnp no)
 		(fields_autoplaced yes)
-		(property "Reference" "#PWR01"
+		(property "Reference" "#PWR0107"
 			(at 144.78 118.11 0)
 			(effects
@@
 				)
 			)
+			(project "fh07_node"
+				(path "/aea54c0a-0593-4c80-97cc-583e63973e87/f7042617-bbaf-4506-802a-37539c441d1d"
+					(reference "#PWR0107")
+					(unit 1)
+				)
+			)
+		)
+	)
+	(symbol
+		(lib_id "power:VCC")
+		(at 144.78 83.82 0)
+		(unit 1)
+		(exclude_from_sim no)
+		(in_bom yes)
+		(on_board yes)
+		(dnp no)
+		(fields_autoplaced yes)
+		(property "Reference" "#PWR0106"
+			(at 144.78 87.63 0)
+			(effects
+				(font
+					(size 1.27 1.27)
+				)
+				(hide yes)
+			)
+		)
+		(property "Value" "VCC"
+			(at 144.78 78.74 0)
+			(effects
+				(font
+					(size 1.27 1.27)
+				)
+			)
+		)
+		(property "Footprint" ""
+			(at 144.78 83.82 0)
+			(effects
+				(font
+					(size 1.27 1.27)
+				)
+				(hide yes)
+			)
+		)
+		(property "Datasheet" ""
+			(at 144.78 83.82 0)
+			(effects
+				(font
+					(size 1.27 1.27)
+				)
+				(hide yes)
+			)
+		)
+		(property "Description" "Power symbol creates a global label with name \"VCC\""
+			(at 144.78 83.82 0)
+			(effects
+				(font
+					(size 1.27 1.27)
+				)
+				(hide yes)
+			)
+		)
+		(pin "1"
+		)
+		(instances
+			(project "sensors"
+				(path "/62bb0011-0a7e-4eb0-868e-e75c2c4b5ec3"
+					(reference "#PWR0101")
+					(unit 1)
+				)
+			)
+			(project "fh07_node"
+				(path "/aea54c0a-0593-4c80-97cc-583e63973e87/f7042617-bbaf-4506-802a-37539c441d1d"
+					(reference "#PWR0106")
+					(unit 1)
+				)
+			)
 		)
 	)
@@
 		(on_board yes)
 		(dnp no)
-		(property "Reference" "R_PULL3"
+		(property "Reference" "R_PULL1"
 			(at 71.628 94.996 0)
 			(effects
@@
 			)
 		)
-		(property "Footprint" ""
+		(property "Footprint" "Resistor_SMD:R_1206_3216Metric_Pad1.30x1.75mm_HandSolder"
 			(at 64.262 92.71 90)
 			(effects
@@
 				(path "/62bb0011-0a7e-4eb0-868e-e75c2c4b5ec3"
 					(reference "R_PULL3")
+					(unit 1)
+				)
+			)
+			(project "fh07_node"
+				(path "/aea54c0a-0593-4c80-97cc-583e63973e87/f7042617-bbaf-4506-802a-37539c441d1d"
+					(reference "R_PULL1")
 					(unit 1)
 				)
@@
 			)
 		)
-		(property "Footprint" "BNO055:LGA28R50P4X10_380X520X100"
+		(property "Footprint" "ProjectFootprintLib:LGA28R50P4X10_380X520X100"
 			(at 124.46 96.52 0)
 			(effects
@@
 				)
 			)
+			(project "fh07_node"
+				(path "/aea54c0a-0593-4c80-97cc-583e63973e87/f7042617-bbaf-4506-802a-37539c441d1d"
+					(reference "U1")
+					(unit 1)
+				)
+			)
 		)
 	)
@@
 		(on_board yes)
 		(dnp no)
-		(property "Reference" "C3"
+		(property "Reference" "C11"
 			(at 159.258 95.25 0)
 			(effects
@@
 			)
 		)
-		(property "Footprint" ""
+		(property "Footprint" "Capacitor_SMD:C_1206_3216Metric_Pad1.33x1.80mm_HandSolder"
 			(at 157.1752 101.6 0)
 			(effects
@@
 				)
 			)
+			(project "fh07_node"
+				(path "/aea54c0a-0593-4c80-97cc-583e63973e87/f7042617-bbaf-4506-802a-37539c441d1d"
+					(reference "C11")
+					(unit 1)
+				)
+			)
 		)
 	)
@@
 		(dnp no)
 		(fields_autoplaced yes)
-		(property "Reference" "#PWR04"
+		(property "Reference" "#PWR0111"
 			(at 97.79 86.36 0)
 			(effects
@@
 				)
 			)
+			(project "fh07_node"
+				(path "/aea54c0a-0593-4c80-97cc-583e63973e87/f7042617-bbaf-4506-802a-37539c441d1d"
+					(reference "#PWR0111")
+					(unit 1)
+				)
+			)
 		)
 	)
@@
 		(dnp no)
 		(fields_autoplaced yes)
-		(property "Reference" "#PWR02"
+		(property "Reference" "#PWR0108"
 			(at 147.32 90.17 0)
 			(effects
@@
 				)
 			)
+			(project "fh07_node"
+				(path "/aea54c0a-0593-4c80-97cc-583e63973e87/f7042617-bbaf-4506-802a-37539c441d1d"
+					(reference "#PWR0108")
+					(unit 1)
+				)
+			)
 		)
 	)
@@
 		(dnp no)
 		(fields_autoplaced yes)
-		(property "Reference" "#PWR06"
+		(property "Reference" "#PWR0109"
 			(at 97.79 106.68 0)
 			(effects
@@
 				)
 			)
+			(project "fh07_node"
+				(path "/aea54c0a-0593-4c80-97cc-583e63973e87/f7042617-bbaf-4506-802a-37539c441d1d"
+					(reference "#PWR0109")
+					(unit 1)
+				)
+			)
 		)
 	)
@@
 		(dnp no)
 		(fields_autoplaced yes)
-		(property "Reference" "#PWR05"
+		(property "Reference" "#PWR0110"
 			(at 97.79 104.14 0)
 			(effects
@@
 				)
 			)
+			(project "fh07_node"
+				(path "/aea54c0a-0593-4c80-97cc-583e63973e87/f7042617-bbaf-4506-802a-37539c441d1d"
+					(reference "#PWR0110")
+					(unit 1)
+				)
+			)
 		)
 	)
@@
 		(dnp no)
 		(fields_autoplaced yes)
-		(property "Reference" "R_PULL4"
+		(property "Reference" "R_PULL2"
 			(at 86.36 86.3599 0)
 			(effects
@@
 			)
 		)
-		(property "Footprint" ""
+		(property "Footprint" "Resistor_SMD:R_1206_3216Metric_Pad1.30x1.75mm_HandSolder"
 			(at 82.042 87.63 90)
 			(effects
@@
 				)
 			)
+			(project "fh07_node"
+				(path "/aea54c0a-0593-4c80-97cc-583e63973e87/f7042617-bbaf-4506-802a-37539c441d1d"
+					(reference "R_PULL2")
+					(unit 1)
+				)
+			)
 		)
 	)
@@
 		(dnp no)
 		(fields_autoplaced yes)
-		(property "Reference" "#PWR03"
+		(property "Reference" "#PWR0112"
 			(at 97.79 83.82 0)
 			(effects
@@
 				)
 			)
-		)
-	)
-	(symbol
-		(lib_id "power:VCC")
-		(at 144.78 83.82 0)
-		(unit 1)
-		(exclude_from_sim no)
-		(in_bom yes)
-		(on_board yes)
-		(dnp no)
-		(fields_autoplaced yes)
-		(property "Reference" "#PWR0101"
-			(at 144.78 87.63 0)
-			(effects
-				(font
-					(size 1.27 1.27)
-				)
-				(hide yes)
-			)
-		)
-		(property "Value" "VCC"
-			(at 144.78 78.74 0)
-			(effects
-				(font
-					(size 1.27 1.27)
-				)
-			)
-		)
-		(property "Footprint" ""
-			(at 144.78 83.82 0)
-			(effects
-				(font
-					(size 1.27 1.27)
-				)
-				(hide yes)
-			)
-		)
-		(property "Datasheet" ""
-			(at 144.78 83.82 0)
-			(effects
-				(font
-					(size 1.27 1.27)
-				)
-				(hide yes)
-			)
-		)
-		(property "Description" "Power symbol creates a global label with name \"VCC\""
-			(at 144.78 83.82 0)
-			(effects
-				(font
-					(size 1.27 1.27)
-				)
-				(hide yes)
-			)
-		)
-		(pin "1"
-		)
-		(instances
-			(project "sensors"
-				(path "/62bb0011-0a7e-4eb0-868e-e75c2c4b5ec3"
-					(reference "#PWR0101")
-					(unit 1)
-				)
+			(project "fh07_node"
+				(path "/aea54c0a-0593-4c80-97cc-583e63973e87/f7042617-bbaf-4506-802a-37539c441d1d"
+					(reference "#PWR0112")
+					(unit 1)
+				)
